File: Bayieeemax_Project.sch (KiCad schematic (older format))
At the start: 16 parts

Commit message: new symbols
Parts:
- A? (x6): symbol Driver_Motor:Pololu_Breakout_DRV8825 -> Bayieeemax_Project-rescue:Pololu_Breakout_DRV8825-Driver_Motor
- M? (x6): symbol Motor:Stepper_Motor_bipolar -> Bayieeemax_Project-rescue:Stepper_Motor_bipolar-Motor
- U?: symbol MCU_ST_STM32F1:STM32F103C8Tx -> Bayieeemax_Project-rescue:STM32F103C8Tx-MCU_ST_STM32F1
- U?: symbol acs712elctr-20a-t:ACS712ELCTR-20A-T -> Bayieeemax_Project-rescue:ACS712ELCTR-20A-T-acs712elctr-20a-t
- VR?: symbol XL4015:XL4015 -> Bayieeemax_Project-rescue:XL4015-XL4015
Changed lines of the file:
@@
 $EndDescr
 $Comp
-L XL4015:XL4015 VR?
+L Bayieeemax_Project-rescue:XL4015-XL4015 VR?
 U 1 1 61931A63
 P 1600 8000
@@
 $EndComp
 $Comp
-L Driver_Motor:Pololu_Breakout_DRV8825 A?
+L Bayieeemax_Project-rescue:Pololu_Breakout_DRV8825-Driver_Motor A?
 U 1 1 6193332A
 P 20350 1750
@@
 $EndComp
 $Comp
-L MCU_ST_STM32F1:STM32F103C8Tx U?
+L Bayieeemax_Project-rescue:STM32F103C8Tx-MCU_ST_STM32F1 U?
 U 1 1 61940A6C
 P 11550 5750
@@
 $EndComp
 $Comp
-L power:+5V #PWR?
+L Bayieeemax_Project-rescue:+5V-power #PWR?
 U 1 1 6194F30C
 P 2100 7800
@@
 $EndComp
 $Comp
-L power:GND #PWR?
+L Bayieeemax_Project-rescue:GND-power #PWR?
 U 1 1 619520C4
 P 1600 8500
@@
 	21500 1350 21500 1300
 $Comp
-L Motor:Stepper_Motor_bipolar M?
+L Bayieeemax_Project-rescue:Stepper_Motor_bipolar-Motor M?
 U 1 1 619340FB
 P 21600 1650
@@
 	21700 2050 21700 1950
 $Comp
-L Driver_Motor:Pololu_Breakout_DRV8825 A?
+L Bayieeemax_Project-rescue:Pololu_Breakout_DRV8825-Driver_Motor A?
 U 1 1 619A8A19
 P 20350 3750
@@
 	21500 3350 21500 3300
 $Comp
-L Motor:Stepper_Motor_bipolar M?
+L Bayieeemax_Project-rescue:Stepper_Motor_bipolar-Motor M?
 U 1 1 619A8A20
 P 21600 3650
@@
 	21700 4050 21700 3950
 $Comp
-L Driver_Motor:Pololu_Breakout_DRV8825 A?
+L Bayieeemax_Project-rescue:Pololu_Breakout_DRV8825-Driver_Motor A?
 U 1 1 619A995D
 P 20400 5550
@@
 	21550 5150 21550 5100
 $Comp
-L Motor:Stepper_Motor_bipolar M?
+L Bayieeemax_Project-rescue:Stepper_Motor_bipolar-Motor M?
 U 1 1 619A9964
 P 21650 5450
@@
 	21750 5850 21750 5750
 $Comp
-L Driver_Motor:Pololu_Breakout_DRV8825 A?
+L Bayieeemax_Project-rescue:Pololu_Breakout_DRV8825-Driver_Motor A?
 U 1 1 619AB0ED
 P 20400 7250
@@
 	21550 6850 21550 6800
 $Comp
-L Motor:Stepper_Motor_bipolar M?
+L Bayieeemax_Project-rescue:Stepper_Motor_bipolar-Motor M?
 U 1 1 619AB0F4
 P 21650 7150
@@
 	2650 1700 2900 1700
 $Comp
-L Motor:Stepper_Motor_bipolar M?
+L Bayieeemax_Project-rescue:Stepper_Motor_bipolar-Motor M?
 U 1 1 619AF0C6
 P 3500 1700
@@
 	3400 1400 3400 1350
 $Comp
-L Driver_Motor:Pololu_Breakout_DRV8825 A?
+L Bayieeemax_Project-rescue:Pololu_Breakout_DRV8825-Driver_Motor A?
 U 1 1 619AF0BF
 P 2250 1800
@@
 $EndComp
 $Comp
-L Driver_Motor:Pololu_Breakout_DRV8825 A?
+L Bayieeemax_Project-rescue:Pololu_Breakout_DRV8825-Driver_Motor A?
 U 1 1 619B004B
 P 2250 3700
@@
 	3400 3300 3400 3250
 $Comp
-L Motor:Stepper_Motor_bipolar M?
+L Bayieeemax_Project-rescue:Stepper_Motor_bipolar-Motor M?
 U 1 1 619B0052
 P 3500 3600
@@
 	3600 4000 3600 3900
 $Comp
-L power:+12V #PWR?
+L Bayieeemax_Project-rescue:+12V-power #PWR?
 U 1 1 61954A0B
 P 1100 7800
@@
 $EndComp
 $Comp
-L power:GND #PWR?
+L Bayieeemax_Project-rescue:GND-power #PWR?
 U 1 1 61964EC6
 P 2250 4500
@@
 $EndComp
 $Comp
-L power:GND #PWR?
+L Bayieeemax_Project-rescue:GND-power #PWR?
 U 1 1 61966167
 P 2350 4500
@@
 $EndComp
 $Comp
-L power:GND #PWR?
+L Bayieeemax_Project-rescue:GND-power #PWR?
 U 1 1 6196B455
 P 2250 2600
@@
 $EndComp
 $Comp
-L power:GND #PWR?
+L Bayieeemax_Project-rescue:GND-power #PWR?
 U 1 1 6196B45B
 P 2350 2600
@@
 $EndComp
 $Comp
-L power:GND #PWR?
+L Bayieeemax_Project-rescue:GND-power #PWR?
 U 1 1 6196E396
 P 20350 2550
@@
 $EndComp
 $Comp
-L power:GND #PWR?
+L Bayieeemax_Project-rescue:GND-power #PWR?
 U 1 1 6196E39C
 P 20450 2550
@@
 $EndComp
 $Comp
-L power:GND #PWR?
+L Bayieeemax_Project-rescue:GND-power #PWR?
 U 1 1 6196FB7F
 P 20350 4550
@@
 $EndComp
 $Comp
-L power:GND #PWR?
+L Bayieeemax_Project-rescue:GND-power #PWR?
 U 1 1 6196FB85
 P 20450 4550
@@
 $EndComp
 $Comp
-L power:GND #PWR?
+L Bayieeemax_Project-rescue:GND-power #PWR?
 U 1 1 619714FC
 P 20400 6350
@@
 $EndComp
 $Comp
-L power:GND #PWR?
+L Bayieeemax_Project-rescue:GND-power #PWR?
 U 1 1 61971502
 P 20500 6350
@@
 $EndComp
 $Comp
-L power:GND #PWR?
+L Bayieeemax_Project-rescue:GND-power #PWR?
 U 1 1 619730A7
 P 20400 8050
@@
 $EndComp
 $Comp
-L power:GND #PWR?
+L Bayieeemax_Project-rescue:GND-power #PWR?
 U 1 1 619730AD
 P 20500 8050
@@
 $EndComp
 $Comp
-L acs712elctr-20a-t:ACS712ELCTR-20A-T U?
+L Bayieeemax_Project-rescue:ACS712ELCTR-20A-T-acs712elctr-20a-t U?
 U 1 1 619E1256
-P 8500 11350
-F 0 "U?" H 8500 12020 50  0000 C CNN
-F 1 "ACS712ELCTR-20A-T" H 8500 11929 50  0000 C CNN
-F 2 "SOIC127P600X175-8N" H 9050 10750 50  0001 L BNN
-F 3 "" H 8500 11350 50  0001 L BNN
-	1    8500 11350
-	1    0    0    -1
-$EndComp
+P 6900 11350
+F 0 "U?" H 6900 12020 50  0000 C CNN
+F 1 "ACS712ELCTR-20A-T" H 6900 11929 50  0000 C CNN
+F 2 "SOIC127P600X175-8N" H 7450 10750 50  0001 L BNN
+F 3 "" H 6900 11350 50  0001 L BNN
+	1    6900 11350
+	1    0    0    -1
+$EndComp

Commit message: Novas alterações
Parts:
- removed A? (x5): Pololu_Breakout_DRV8825, Module:Pololu_Breakout-16_15.2x20.3mm, symbol Bayieeemax_Project-rescue:Pololu_Breakout_DRV8825-Driver_Motor
- removed M? (x6): Stepper_Motor_bipolar, symbol Bayieeemax_Project-rescue:Stepper_Motor_bipolar-Motor
- removed U?: STM32F103C8Tx, Package_QFP:LQFP-48_7x7mm_P0.5mm, symbol Bayieeemax_Project-rescue:STM32F103C8Tx-MCU_ST_STM32F1
- removed U?: Módulo_GPS_VK2828U7G5LF_TTL, symbol Baiyeeemax:Módulo_GPS_VK2828U7G5LF_TTL
- removed U?: ACS712ELCTR-20A-T, SOIC127P600X175-8N, symbol Bayieeemax_Project-rescue:ACS712ELCTR-20A-T-acs712elctr-20a-t
- added C?: 100uF, symbol Device:C
- added J?: Raspberry_POWER_IN, symbol Connector_Generic:Conn_01x02
- added J?: ACS_SENSOR, symbol Connector_Generic:Conn_01x03
- added J?: USB_TTL, symbol Connector_Generic:Conn_01x06
- added J?: Motor1, symbol Connector_Generic:Conn_01x04
- added J?: Baterry_P.IN, symbol Connector_Generic:Conn_01x02
- added R?: 1.7K, symbol Device:R
- added R?: 3.3K, symbol Device:R
- added U?: ChinaBluePill, symbol Bayieeemax_Project-rescue:ChinaBluePill
- A?: value Pololu_Breakout_DRV8825 -> Pololu_Breakout_DRV8825_1
Connections:
- net labels added: +3V3, ACS, Direction_1, MOTOR1_A1, MOTOR1_A2, MOTOR1_B1, MOTOR1_B2, Reset_1, Rx_SERIAL, Tx_SERIAL
- wire segments 48 -> 46
- no-connect marks 0 -> 7
Other:
- note added: "USB_Raspbery_charge\n"
- moved on the sheet: A?, VR?

Commit message: edicoes
Parts:
- added A?: Pololu_Breakout_DRV8825_2, Module:Pololu_Breakout-16_15.2x20.3mm, symbol Bayieeemax_Project-rescue:Pololu_Breakout_DRV8825-Driver_Motor
- added A?: Pololu_Breakout_DRV8825_3, Module:Pololu_Breakout-16_15.2x20.3mm, symbol Bayieeemax_Project-rescue:Pololu_Breakout_DRV8825-Driver_Motor
- added A?: Pololu_Breakout_DRV8825_4, Module:Pololu_Breakout-16_15.2x20.3mm, symbol Bayieeemax_Project-rescue:Pololu_Breakout_DRV8825-Driver_Motor
- added A?: Pololu_Breakout_DRV8825_5, Module:Pololu_Breakout-16_15.2x20.3mm, symbol Bayieeemax_Project-rescue:Pololu_Breakout_DRV8825-Driver_Motor
- added A?: Pololu_Breakout_DRV8825_6, Module:Pololu_Breakout-16_15.2x20.3mm, symbol Bayieeemax_Project-rescue:Pololu_Breakout_DRV8825-Driver_Motor
- added C?: 1000uF, symbol Device:C
- added C? (x5): 100uF, symbol Device:C
- added J?: STP_RESOL/POWER_1, symbol Connector_Generic:Conn_02x03_Odd_Even
- added J?: GPS_Conn, symbol Connector_Generic:Conn_01x06
- added J?: Motor2, symbol Connector_Generic:Conn_01x04
- added J?: STP_RESOL/POWER_2, symbol Connector_Generic:Conn_02x03_Odd_Even
- added J?: Motor3, symbol Connector_Generic:Conn_01x04
- added J?: STP_RESOL/POWER_3, symbol Connector_Generic:Conn_02x03_Odd_Even
- added J?: Motor4, symbol Connector_Generic:Conn_01x04
- added J?: STP_RESOL/POWER_4, symbol Connector_Generic:Conn_02x03_Odd_Even
- added J?: Motor5, symbol Connector_Generic:Conn_01x04
- added J?: STP_RESOL/POWER_5, symbol Connector_Generic:Conn_02x03_Odd_Even
- added J?: Motor6, symbol Connector_Generic:Conn_01x04
- added J?: STP_RESOL/POWER_6, symbol Connector_Generic:Conn_02x03_Odd_Even
- added J?: TTL_Raspberry, symbol Connector_Generic:Conn_01x02
- added J?: Conn_01x06_Female, symbol Connector:Conn_01x06_Female
- added J?: I2C_MPU_Raspberry, symbol Connector_Generic:Conn_01x02
- added J?: I2C_MAX30100_Raspberry, symbol Connector_Generic:Conn_01x02
- added J?: MAX300100_Conn, symbol Connector:Conn_01x07_Female
- added U?: MPU-9250, QFN40P300X300X105-24N, symbol Bayieeemax_Project-rescue:MPU-9250
- added U?: MAX30100EFD+, LGA14R80P2X7_560X280X130, symbol Bayieeemax_Project-rescue:MAX30100EFD+
Connections:
- net labels added: +15V, +3.3V, ADO_MPU9250, DIREC_1, DIREC_2, DIREC_3, DIREC_4, DIREC_5, DIREC_6, EN_GPS, GND_GPS, IRO, M0_1, M0_2, M0_3, M0_4, M0_5, M0_6, M1_1, M1_2, M1_3, M1_4, M1_5, M1_6, M2_1, M2_2, M2_3, M2_4, M2_5, M2_6, MOTOR2_A1, MOTOR2_A2, MOTOR2_B1, MOTOR2_B2, MOTOR3_A1, MOTOR3_A2, MOTOR3_B1, MOTOR3_B2, MOTOR4_A1, MOTOR4_A2, MOTOR4_B1, MOTOR4_B2, MOTOR5_A1, MOTOR5_A2, MOTOR5_B1, MOTOR5_B2, MOTOR6_A1, MOTOR6_A2, MOTOR6_B1, MOTOR6_B2, PPS_GPS, RD, RX_GPS, SCL_MAX3100, SDA_MAX3100, SDA_MPU9250, SLC_MPU9250, STEP_1, STEP_2, STEP_3, STEP_4, STEP_5, STEP_6, TX_GPS, VCC3V3_GPS, nCS_MPU9250, ~INT
- net labels removed: +12V, Direction_1, Reset_1
- wire segments 46 -> 273
- no-connect marks 7 -> 20
Other:
- moved on the sheet: A?, C?, J?, R?, VR?

Commit message: eeschema edicoes
Parts:
- removed J?: Conn_01x06_Female, symbol Connector:Conn_01x06_Female
- removed J?: I2C_MAX30100_Raspberry, symbol Connector_Generic:Conn_01x02
- removed J?: MAX300100_Conn, symbol Connector:Conn_01x07_Female
- removed U?: MAX30100EFD+, LGA14R80P2X7_560X280X130, symbol Bayieeemax_Project-rescue:MAX30100EFD+
- added J?: I2C_MAX30100_Raspberry, symbol Connector_Generic:Conn_01x02
- added U?: MAX30100EFD+, LGA14R80P2X7_560X280X130, symbol Bayieeemax_Project-rescue:MAX30100EFD+
Connections:
- net labels removed: ADO_MPU9250, nCS_MPU9250
- wire segments 273 -> 265
- no-connect marks 20 -> 31
Other:
- note added: "5V pwm tolerant\n"
- note added: "UART GPS\n\n"
- moved on the sheet: J?, R?, U?, VR?

Commit message: V01 do circuito
Parts:
- removed J?: STP_RESOL/POWER_1, symbol Connector_Generic:Conn_02x03_Odd_Even
- removed J?: STP_RESOL/POWER_2, symbol Connector_Generic:Conn_02x03_Odd_Even
- removed J?: STP_RESOL/POWER_3, symbol Connector_Generic:Conn_02x03_Odd_Even
- removed J?: STP_RESOL/POWER_4, symbol Connector_Generic:Conn_02x03_Odd_Even
- removed J?: STP_RESOL/POWER_5, symbol Connector_Generic:Conn_02x03_Odd_Even
- removed J?: STP_RESOL/POWER_6, symbol Connector_Generic:Conn_02x03_Odd_Even
- added J10: MicroStep_1/32, symbol Connector_Generic:Conn_02x03_Odd_Even
- added J9: MicroStep_1/16, symbol Connector_Generic:Conn_02x03_Odd_Even
- gave numbers to parts that had none: 33
Connections:
- net labels added: +3V0, M0, M1, M2
- net labels removed: IRO, M0_1, M0_2, M0_3, M0_4, M0_5, M0_6, M1_1, M1_2, M1_3, M1_4, M1_5, M1_6, M2_1, M2_2, M2_3, M2_4, M2_5, M2_6, RD, ~INT
- wire segments 265 -> 232
- no-connect marks 31 -> 35
Other:
- moved on the sheet: J6, J7

Commit message: New files
Parts:
- removed U3: MAX30100EFD+, LGA14R80P2X7_560X280X130, symbol Bayieeemax_Project-rescue:MAX30100EFD+
- added C8: 100nf, Capacitor_SMD:C_Elec_6.3x7.7, symbol Device:C
- added J17: i2C_MAX30100, Connector_PinSocket_2.54mm:PinSocket_1x06_P2.54mm_Vertical, symbol Connector_Generic:Conn_01x07
- added R3, R4: 10K, Resistor_THT:R_Axial_DIN0207_L6.3mm_D2.5mm_P10.16mm_Horizontal, symbol Device:R
- C1: footprint (none) -> Capacitor_THT:C_Radial_D10.0mm_H12.5mm_P5.00mm
- C2, C3, C4, C5, C6, C7: footprint (none) -> Capacitor_SMD:C_Elec_6.3x7.7
- J1, J3: footprint (none) -> Baiyeeemax:TerminalBlock_Phoenix_PT-1,5-2-5.0-H_1x02_P5.00mm_Horizontal
- J10, J9: footprint (none) -> Connector_PinHeader_2.00mm:PinHeader_2x03_P2.00mm_Vertical
- J11, J12, J13, J14, J15, J16: footprint (none) -> Connector_PinHeader_2.00mm:PinHeader_1x04_P2.00mm_Vertical
- J2: footprint (none) -> Connector_PinHeader_2.54mm:PinHeader_1x06_P2.54mm_Vertical
- J4: footprint (none) -> Connector_PinHeader_2.54mm:PinHeader_1x03_P2.54mm_Vertical
- J5, J7, J8: footprint (none) -> Connector_PinHeader_2.54mm:PinHeader_1x02_P2.54mm_Vertical
- J6: footprint (none) -> Connector_Molex:Molex_MicroClasp_55935-0630_1x06_P2.00mm_Horizontal
- R1, R2: footprint (none) -> Resistor_THT:R_Axial_DIN0207_L6.3mm_D2.5mm_P10.16mm_Horizontal
- U1: footprint QFN40P300X300X105-24N -> Baiyeeemax:QFN40P300X300X105-24N
- U2: footprint (none) -> Baiyeeemax:BluePill_STM32F103C
- VR1: footprint CONV_XL4015 -> Baiyeeemax:DCDC_stepdown_75W-XL4015
Connections:
- net labels added: ~INT_MAX3100
- net labels removed: +3V0, EN_GPS, GND_GPS, PPS_GPS, VCC3V3_GPS
- wire segments 232 -> 254
- no-connect marks 35 -> 47
Other:
- note added: "En"
- note added: "GND\n"
- note added: "Microcontroller\n"
- note added: "Power_source\n"
- note added: "Sensors\n"
- note added: "Step Motor + Drivers + Step Mode\n"
- note added: "VCC3.3V\n"
- note removed: "5V pwm tolerant\n"
- moved on the sheet: J2, J3, J4, J5, J7, J8, R1, R2, U1, U2, VR1

Commit message: Changes
Parts:
- added J18: Raspberry_POWER_IN, Baiyeeemax:TerminalBlock_Phoenix_PT-1,5-2-5.0-H_1x02_P5.00mm_Horizontal, symbol Connector_Generic:Conn_01x02
- added R5: 13K, Resistor_THT:R_Axial_DIN0207_L6.3mm_D2.5mm_P10.16mm_Horizontal, symbol Device:R
- added R6: 3K, Resistor_THT:R_Axial_DIN0207_L6.3mm_D2.5mm_P10.16mm_Horizontal, symbol Device:R
- J3: value Raspberry_POWER_IN -> Current_power_in
- U1: footprint Baiyeeemax:QFN40P300X300X105-24N -> Baiyeeemax:MPU-9250
Connections:
- net +15V: no longer C1.2, J1.1 (Pin_1), VR1.5 (VIN)
- net +5V: now also J18.1 (Pin_1); no longer J3.1 (Pin_1)
- net GND: now also J18.2 (Pin_2), R6.2; no longer J3.2 (Pin_2)
- net ~INT_MAX3100: now also U2.13 (PB5)
- net AVS: now reaches U2.15 (PB7)
- net AVS: now also R5.2, R6.1
- new net: J1.1 (Pin_1), J3.2 (Pin_2)
- new net +12V: C1.2, J3.1 (Pin_1), R5.1, VR1.5 (VIN)
- no-connect marks 47 -> 45
Other:
- moved on the sheet: C1, J1, J8, VR1

Commit message: changes
Parts:
- removed A5: Pololu_Breakout_DRV8825_5, Module:Pololu_Breakout-16_15.2x20.3mm, symbol Bayieeemax_Project-rescue:Pololu_Breakout_DRV8825-Driver_Motor
- removed A6: Pololu_Breakout_DRV8825_6, Module:Pololu_Breakout-16_15.2x20.3mm, symbol Bayieeemax_Project-rescue:Pololu_Breakout_DRV8825-Driver_Motor
- removed C6, C7: 100uF, Capacitor_SMD:C_Elec_6.3x7.7, symbol Device:C
- removed J15: Motor5, Connector_PinHeader_2.00mm:PinHeader_1x04_P2.00mm_Vertical, symbol Connector_Generic:Conn_01x04
- removed J16: Motor6, Connector_PinHeader_2.00mm:PinHeader_1x04_P2.00mm_Vertical, symbol Connector_Generic:Conn_01x04
- C2, C3, C4, C5: footprint Capacitor_SMD:C_Elec_6.3x7.7 -> Baiyeeemax:CP_Radial_D6.3mm_P2.50mm
- C8: footprint Capacitor_SMD:C_Elec_6.3x7.7 -> Capacitor_THT:C_Disc_D7.5mm_W2.5mm_P5.00mm
- J10: value MicroStep_1/32 -> MicroStep_1/32_wheels
- J6: footprint Connector_Molex:Molex_MicroClasp_55935-0630_1x06_P2.00mm_Horizontal -> Connector_PinSocket_2.54mm:PinSocket_1x06_P2.54mm_Vertical
- J9: value MicroStep_1/16 -> MicroStep_1/16_wheels
Connections:
- net DIREC_6 is gone; now on net DIREC_4: U2.1 (PB12)
- net DIREC_4: no longer U2.2 (PB13)
- net DIREC_5: no longer names the net of U2.3 (PB14)
- net STEP_5: no longer names the net of U2.34 (PB1)
- net STEP_6: no longer names the net of U2.33 (PB0)
