File: Bayieeemax_Project.sch (KiCad schematic (older format))
At the start: 35 parts, among them J1 Baterry_P.IN, J10 MicroStep_1/32_wheels, J11 Motor1, J12 Motor2, J13 Motor3, J14 Motor4, J17 i2C_MAX30100, J18 Raspberry_POWER_IN, J2 USB_TTL, J3 Current_power_in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

Commit message: Board
Parts:
- J17: footprint Connector_PinSocket_2.54mm:PinSocket_1x06_P2.54mm_Vertical -> Baiyeeemax:MAX30100
Connections:
- net ACS: now also U2.30 (PA5); no longer U2.14 (PB6)
- net AVS: now also U2.31 (PA6); no longer U2.15 (PB7)
- net SDA_MPU9250: now also U2.15 (PB7)
- net SLC_MPU9250: now also U2.14 (PB6)
- no-connect marks 45 -> 34
Changed lines of the file:
@@
 	1    0    0    -1
 $EndComp
-NoConn ~ 6900 9850
-NoConn ~ 6900 9750
 Wire Wire Line
 	8500 8850 8600 8850
@@
 Text Label 6800 9450 2    50   ~ 0
 SLC_MPU9250
-$Comp
-L Bayieeemax_Project-rescue:MPU-9250 U1
-U 1 1 61C9EC7E
-P 7700 9550
-F 0 "U1" H 7700 10515 50  0000 C CNN
-F 1 "MPU-9250" H 7700 10424 50  0000 C CNN
-F 2 "Baiyeeemax:MPU-9250" H 7750 10350 50  0001 L BNN
-F 3 "" H 7800 9850 50  0001 L BNN
-F 4 "MPU-9250" H 7300 10350 50  0001 L BNN "MP"
-F 5 "SMD Gyroscope/Accelerometer/Magnetometer Sensor; 9-AXIS" H 7200 8600 50  0001 L BNN "DESCRIPTION"
-F 6 "The center Exposed Pad (EP), for MPU devices is a No Connect (NC) pad. To avoid package stress, do not solder the EP to the PCB. Please refer to the document “AN-IVS-0002A-00”. As a result of these guidelines, the exposed pad has not been included on the PCB footprint. We’ve added a keep-out area under the exposed pad. Please don’t route traces or vias under the part, on the same side of the board" H 5750 11200 50  0001 L BNN "NOTES"
-	1    7700 9550
-	1    0    0    -1
-$EndComp
 Wire Wire Line
 	13300 9550 13250 9550
@@
 	10700 5600 10750 5600
 NoConn ~ 6900 9650
-NoConn ~ 6900 9150
-NoConn ~ 8500 8950
-NoConn ~ 8500 9150
-NoConn ~ 8500 9350
-NoConn ~ 8500 9550
-NoConn ~ 8500 9650
-NoConn ~ 8500 9750
 NoConn ~ 6900 9350
 Text Label 20400 1700 2    50   ~ 0
@@
 NoConn ~ 9300 4900
 NoConn ~ 9300 5000
-NoConn ~ 9300 5500
 NoConn ~ 10700 6300
 NoConn ~ 10700 6400
@@
 	10750 6000 10700 6000
 NoConn ~ 9300 5300
-NoConn ~ 9300 5400
 NoConn ~ 10750 5100
 NoConn ~ 10750 5200
@@
 Microcontroller\n
 Wire Notes Line
-	5850 8400 15000 8400
-Wire Notes Line
-	15000 8400 15000 12150
-Wire Notes Line
 	15000 12150 5850 12150
 Wire Notes Line
@@
 F 0 "J17" H 12130 9942 50  0000 L CNN
 F 1 "i2C_MAX30100" H 11950 9500 50  0000 L CNN
-F 2 "Connector_PinSocket_2.54mm:PinSocket_1x06_P2.54mm_Vertical" H 12050 9900 50  0001 C CNN
+F 2 "Baiyeeemax:MAX30100" H 12050 9900 50  0001 C CNN
 F 3 "~" H 12050 9900 50  0001 C CNN
 	1    12050 9900
@@
 	11800 9600 11850 9600
 Connection ~ 11800 9200
-Text Label 10950 5400 2    50   ~ 0
+Text Label 9250 5400 2    50   ~ 0
 ACS
-Wire Wire Line
-	10700 5400 10950 5400
 Text Notes 7450 11350 0    50   ~ 0
 USB_Raspbery_charge\n
@@
 	2950 2250 2950 2450
 Connection ~ 2950 2450
-Text Label 10800 5500 0    50   ~ 0
+Text Label 9250 5500 2    50   ~ 0
 AVS
-Wire Wire Line
-	10700 5500 10800 5500
 $Comp
 L Bayieeemax_Project-rescue:+16.8V #PWR0107
@@
 NoConn ~ 10700 6100
 NoConn ~ 10700 6200
+Text Label 10750 5500 0    50   ~ 0
+SDA_MPU9250
+Text Label 10750 5400 0    50   ~ 0
+SLC_MPU9250
+Wire Wire Line
+	9250 5500 9300 5500
+Wire Wire Line
+	9300 5400 9250 5400
+Wire Wire Line
+	10700 5400 10750 5400
+Wire Wire Line
+	10750 5500 10700 5500
+$Comp
+L Bayieeemax_Project-rescue:MPU-9250 U1
+U 1 1 61C9EC7E
+P 7700 9550
+F 0 "U1" H 7700 10515 50  0000 C CNN
+F 1 "MPU-9250" H 7700 10424 50  0000 C CNN
+F 2 "Baiyeeemax:MPU-9250" H 7750 10350 50  0001 L BNN
+F 3 "" H 7800 9850 50  0001 L BNN
+F 4 "MPU-9250" H 7300 10350 50  0001 L BNN "MP"
+F 5 "SMD Gyroscope/Accelerometer/Magnetometer Sensor; 9-AXIS" H 7200 8600 50  0001 L BNN "DESCRIPTION"
+F 6 "The center Exposed Pad (EP), for MPU devices is a No Connect (NC) pad. To avoid package stress, do not solder the EP to the PCB. Please refer to the document “AN-IVS-0002A-00”. As a result of these guidelines, the exposed pad has not been included on the PCB footprint. We’ve added a keep-out area under the exposed pad. Please don’t route traces or vias under the part, on the same side of the board" H 5750 11200 50  0001 L BNN "NOTES"
+	1    7700 9550
+	1    0    0    -1
+$EndComp
+Wire Notes Line
+	15000 8400 15000 12150
+Wire Notes Line
+	5850 8400 15000 8400
 $EndSCHEMATC
