File: Bayieeemax_Project.kicad_pcb (KiCad board)
At the start: 2 copper layers, 50 x 50 mm, 38 parts, among them J1 Baterry_P.IN, J10 MicroStep_1/32, J11 Motor1, J12 Motor2, J13 Motor3, J14 Motor4, J15 Motor5, J16 Motor6, J17 i2C_MAX30100, J2 USB_TTL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

Commit message: Changes
Parts:
- added J18: Raspberry_POWER_IN, Baiyeeemax:TerminalBlock_Phoenix_PT-1,5-2-5.0-H_1x02_P5.00mm_Horizontal, F.Cu at (194.5, 80.6)
- added R5: 13K, Resistor_THT:R_Axial_DIN0207_L6.3mm_D2.5mm_P10.16mm_Horizontal, F.Cu at (192.6, 73.6)
- added R6: 3K, Resistor_THT:R_Axial_DIN0207_L6.3mm_D2.5mm_P10.16mm_Horizontal, F.Cu at (205.9, 73.6)
- J3: value Raspberry_POWER_IN -> Current_power_in
- U1: footprint Baiyeeemax:QFN40P300X300X105-24N -> Baiyeeemax:MPU-9250
- moved J13 122.5 mm to (143.9, 112.4)
- moved A3 120.9 mm to (110.3, 116.9)
- moved A2 120.9 mm to (127.1, 116.9)
- moved J16 109.4 mm to (161.9, 124.2)
- moved C8 84.0 mm to (168.9, 134.4)
- moved A4 78.1 mm to (93.6, 116.9)
- moved J2 74.5 mm to (144.2, 95.3)
- moved U1 72.7 mm to (183.4, 75.6)
- moved C6 72.2 mm to (187.8, 111.8)
- moved J9 70.1 mm to (212.7, 87.7)
- moved C4 70.0 mm to (168.9, 126.3)
- moved A1 68.6 mm to (93.6, 95.0)
- moved C2 52.2 mm to (192.3, 101.8)
- moved J17 50.3 mm to (173.6, 69.8)
- moved J10 46.5 mm to (175.9, 126.1)
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Connections:
- C1 pad 2: +15V -> +12V
- J1 pad 1: +15V -> Net-(J1-Pad1)
- J3 pad 1: +5V -> +12V
- J3 pad 2: GND -> Net-(J1-Pad1)
- U2 pad 13: Net-(U2-Pad13) -> /~INT_MAX3100
- U2 pad 15: Net-(U2-Pad15) -> /AVS
Other:
- board outline removed

Commit message: changes
Parts:
- removed A5: Pololu_Breakout_DRV8825_5, Module:Pololu_Breakout-16_15.2x20.3mm
- removed A6: Pololu_Breakout_DRV8825_6, Module:Pololu_Breakout-16_15.2x20.3mm
- removed C6, C7: 100uF, Capacitor_SMD:C_Elec_6.3x7.7
- removed J15: Motor5, Connector_PinHeader_2.00mm:PinHeader_1x04_P2.00mm_Vertical
- removed J16: Motor6, Connector_PinHeader_2.00mm:PinHeader_1x04_P2.00mm_Vertical
- C2, C3, C4, C5: footprint Capacitor_SMD:C_Elec_6.3x7.7 -> Baiyeeemax:CP_Radial_D6.3mm_P2.50mm
- C8: footprint Capacitor_SMD:C_Elec_6.3x7.7 -> Capacitor_THT:C_Disc_D7.5mm_W2.5mm_P5.00mm
- J10: value MicroStep_1/32 -> MicroStep_1/32_wheels
- J6: footprint Connector_Molex:Molex_MicroClasp_55935-0630_1x06_P2.00mm_Horizontal -> Connector_PinSocket_2.54mm:PinSocket_1x06_P2.54mm_Vertical
- J9: value MicroStep_1/16 -> MicroStep_1/16_wheels
- moved J5 110.8 mm to (100.5, 116.2)
- moved R5 109.4 mm to (95.1, 123.2)
- moved R6 106.3 mm to (108.4, 115.9)
- moved J8 99.6 mm to (95.8, 116.2)
- moved R3 98.1 mm to (108.4, 119.9)
- moved R4 96.1 mm to (121.7, 115.9)
- moved R1 88.0 mm to (95.1, 128.0)
- moved J18 82.5 mm to (123.6, 122.9)
- moved J6 76.2 mm to (197.0, 68.8)
- moved J9 75.8 mm to (146.2, 124.2)
- moved R2 72.5 mm to (108.4, 124.0)
- moved A2 68.3 mm to (175.3, 68.5)
- moved J14 65.3 mm to (145.9, 94.0)
- moved C8 60.4 mm to (108.8, 128.0)
- moved J11 58.3 mm to (146.2, 114.1)
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Connections:
- U2 pad 1: /DIREC_6 -> /DIREC_4
- U2 pad 2: /DIREC_4 -> Net-(U2-Pad2)
- U2 pad 3: /DIREC_5 -> Net-(U2-Pad3)
- U2 pad 33: /STEP_6 -> Net-(U2-Pad33)
- U2 pad 34: /STEP_5 -> Net-(U2-Pad34)

Commit message: Board
Parts:
- added REF**: MountingHole_3.5mm, MountingHole:MountingHole_3.5mm, F.Cu at (193.0, 124.0)
- added REF**: MountingHole_3.5mm, MountingHole:MountingHole_3.5mm, F.Cu at (92.0, 124.0)
- added REF**: MountingHole_3.5mm, MountingHole:MountingHole_3.5mm, F.Cu at (92.0, 42.0)
- added REF**: MountingHole_3.5mm, MountingHole:MountingHole_3.5mm, F.Cu at (193.0, 42.0)
- J17: footprint Connector_PinSocket_2.54mm:PinSocket_1x06_P2.54mm_Vertical -> Baiyeeemax:MAX30100
- moved R3 109.3 mm to (189.5, 46.8), turned to 270 degrees
- moved J8 107.6 mm to (190.8, 65.5)
- moved C2 100.4 mm to (105.2, 48.8), turned to 180 degrees
- moved J3 97.7 mm to (101.0, 120.0)
- moved J5 96.4 mm to (190.8, 82.2)
- moved R4 94.1 mm to (185.2, 46.5), turned to 270 degrees
- moved R1 92.0 mm to (174.2, 81.2), turned to 90 degrees
- moved C4 89.1 mm to (105.2, 75.2), turned to 180 degrees
- moved C3 85.4 mm to (128.5, 49.0), turned to 180 degrees
- moved J9 78.3 mm to (114.2, 52.8)
- moved J11 78.2 mm to (91.8, 58.0), turned to 180 degrees
- moved R2 74.4 mm to (169.2, 81.2), turned to 90 degrees
- moved J18 68.8 mm to (187.8, 98.0), turned to 90 degrees
- moved J12 68.0 mm to (138.8, 58.0), turned to 180 degrees
- moved C1 60.3 mm to (117.5, 98.2), turned to 180 degrees
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Connections:
- U2 pad 14: /ACS -> /SLC_MPU9250
- U2 pad 15: /AVS -> /SDA_MPU9250
- U2 pad 30: Net-(U2-Pad30) -> /ACS
- U2 pad 31: Net-(U2-Pad31) -> /AVS
Other:
- board outline added: 109 x 90 mm
